File: perception-array-interface-box.kicad_pcb (KiCad board)
At the start: 2 copper layers, 162 x 148 mm, 35 parts, among them J1 PV-3, J2 PV-3, J3 PV-3, J4 2-5530843-7, J5 2-5530843-7, J6 Conn_01x02, J7 RJHSE5381, J8 1715789, U1 K7805-2000R3, U2 K7812-2000R3L

Commit message: Update pcb layout
Parts:
- moved J1 25.4 mm to (127.1, 144.9)
- moved J2 12.7 mm to (101.7, 144.9)
- moved J3 12.7 mm to (114.4, 144.9)
- turned R1 to 180 degrees
Routing:
- net Net-(J2-Pad1): track 6.11 -> 17.2 mm
- net Net-(C1-Pad1): track 39.0 -> 38.3 mm
- net GND: vias 379 -> 373
Changed lines of the file:
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@@
     (thickness 1.6)
     (drawings 54)
-    (tracks 423)
+    (tracks 420)
     (zones 0)
     (modules 35)
@@
   )
   (module Terminal:PV-3_via (layer F.Cu)
-    (at 127.14 144.92)
+    (at 114.44 144.92)
     (fp_text reference J3 (at -2.032 5.08) (layer F.SilkS)
       (effects (font (size 1 1) (thickness 0.15)))
@@
   )
   (module Terminal:PV-3 (layer F.Cu)
-    (at 114.44 144.92)
+    (at 101.74 144.92)
     (fp_text reference J2 (at -2.032 5.08) (layer F.SilkS)
       (effects (font (size 1 1) (thickness 0.15)))
@@
   )
   (module Terminal:PV-3 (layer F.Cu)
-    (at 101.74 144.92)
+    (at 127.14 144.92)
     (fp_text reference J1 (at -2.032 5.08) (layer F.SilkS)
       (effects (font (size 1 1) (thickness 0.15)))
@@
     (fp_line (start 3.81 3.81) (end -3.81 3.81) (layer F.CrtYd) (width 0.12))
     (fp_line (start -3.81 3.81) (end -3.81 -3.81) (layer F.CrtYd) (width 0.12))
-    (fp_text user 24V (at 0 -5.715) (layer F.SilkS)
+    (fp_text user V+ (at 0 -5.715) (layer F.SilkS)
       (effects (font (size 2 2) (thickness 0.15)))
     )
@@
   )
   (module Resistor_SMD:R_0603_1608Metric_Pad1.05x0.95mm_HandSolder (layer F.Cu)
-    (at 114.44 152.54 90)
+    (at 114.44 152.54 180)
     (descr "Resistor SMD 0603 (1608 Metric), square (rectangular) end terminal, IPC_7351 nominal with elongated pad for handsoldering. (Body size source: http://www.tortai-tech.com/upload/download/2011102023233369053.pdf), generated with kicad-footprint-generator")
     (tags "resistor handsolder")
     (attr smd)
-    (fp_text reference R1 (at 0 -1.43 90) (layer F.SilkS)
-      (effects (font (size 1 1) (thickness 0.15)))
-    )
-    (fp_text value 1k (at 0 1.43 90) (layer F.Fab)
+    (fp_text reference R1 (at 0 -1.43) (layer F.SilkS)
+      (effects (font (size 1 1) (thickness 0.15)))
+    )
+    (fp_text value 1k (at 0 1.43) (layer F.Fab)
       (effects (font (size 1 1) (thickness 0.15)))
     )
@@
     (fp_line (start -0.8 -0.4) (end 0.8 -0.4) (layer F.Fab) (width 0.1))
     (fp_line (start -0.8 0.4) (end -0.8 -0.4) (layer F.Fab) (width 0.1))
-    (fp_text user %R (at 0 0 90) (layer F.Fab)
+    (fp_text user %R (at 0 0) (layer F.Fab)
       (effects (font (size 0.4 0.4) (thickness 0.06)))
     )
-    (pad 2 smd roundrect (at 0.875 0 90) (size 1.05 0.95) (layers F.Cu F.Paste F.Mask) (roundrect_rratio 0.25)
+    (pad 2 smd roundrect (at 0.875 0 180) (size 1.05 0.95) (layers F.Cu F.Paste F.Mask) (roundrect_rratio 0.25)
       (net 8 "Net-(J2-Pad1)"))
-    (pad 1 smd roundrect (at -0.875 0 90) (size 1.05 0.95) (layers F.Cu F.Paste F.Mask) (roundrect_rratio 0.25)
+    (pad 1 smd roundrect (at -0.875 0 180) (size 1.05 0.95) (layers F.Cu F.Paste F.Mask) (roundrect_rratio 0.25)
       (net 1 GND))
     (model ${KISYS3DMOD}/Resistor_SMD.3dshapes/R_0603_1608Metric.wrl
@@
   (via (at 111.9 175.4) (size 0.8) (drill 0.4) (layers F.Cu B.Cu) (net 1))
   (via (at 124.6 181.75) (size 0.8) (drill 0.4) (layers F.Cu B.Cu) (net 1))
-  (via (at 130.95 124.6) (size 0.8) (drill 0.4) (layers F.Cu B.Cu) (net 1))
-  (via (at 130.95 137.3) (size 0.8) (drill 0.4) (layers F.Cu B.Cu) (net 1))
-  (via (at 130.95 143.65) (size 0.8) (drill 0.4) (layers F.Cu B.Cu) (net 1))
-  (via (at 130.95 130.95) (size 0.8) (drill 0.4) (layers F.Cu B.Cu) (net 1))
-  (via (at 130.95 118.25) (size 0.8) (drill 0.4) (layers F.Cu B.Cu) (net 1))
-  (via (at 130.95 105.55) (size 0.8) (drill 0.4) (layers F.Cu B.Cu) (net 1))
-  (via (at 130.95 99.2) (size 0.8) (drill 0.4) (layers F.Cu B.Cu) (net 1))
-  (via (at 130.95 92.85) (size 0.8) (drill 0.4) (layers F.Cu B.Cu) (net 1))
   (via (at 137.3 143.65) (size 0.8) (drill 0.4) (layers F.Cu B.Cu) (net 1))
   (via (at 137.3 137.3) (size 0.8) (drill 0.4) (layers F.Cu B.Cu) (net 1))
@@
   (via (at 188.1 213.5) (size 0.8) (drill 0.4) (layers F.Cu B.Cu) (net 1))
   (via (at 194.45 213.5) (size 0.8) (drill 0.4) (layers F.Cu B.Cu) (net 1))
-  (segment (start 106.185 153.175) (end 107.455 154.445) (width 2.54) (layer F.Cu) (net 2))
-  (segment (start 90.31 153.175) (end 106.185 153.175) (width 2.54) (layer F.Cu) (net 2))
-  (segment (start 90.31 148.34) (end 90.31 153.175) (width 2.54) (layer F.Cu) (net 2))
+  (via (at 99.2 150) (size 0.8) (drill 0.4) (layers F.Cu B.Cu) (net 1))
+  (via (at 105.55 150) (size 0.8) (drill 0.4) (layers F.Cu B.Cu) (net 1))
   (segment (start 113.17 160.795) (end 107.455 160.795) (width 2.54) (layer F.Cu) (net 2))
   (segment (start 107.455 160.795) (end 107.455 165.24) (width 2.54) (layer F.Cu) (net 2))
-  (segment (start 107.455 154.445) (end 107.455 160.795) (width 2.54) (layer F.Cu) (net 2))
+  (segment (start 107.455 155.715) (end 107.455 160.795) (width 2.54) (layer F.Cu) (net 2))
+  (segment (start 90.31 153.175) (end 104.915 153.175) (width 2.54) (layer F.Cu) (net 2))
+  (segment (start 90.31 148.34) (end 90.31 153.175) (width 2.54) (layer F.Cu) (net 2))
+  (segment (start 107.455 155.715) (end 104.915 153.175) (width 2.54) (layer F.Cu) (net 2))
   (segment (start 81.42 158.39) (end 81.42 148.34) (width 2.54) (layer F.Cu) (net 3))
   (segment (start 79.515 170.32) (end 81.42 168.415) (width 2.54) (layer F.Cu) (net 3))
@@
   (segment (start 79.515 175.4) (end 81.42 177.305) (width 2.54) (layer F.Cu) (net 6))
   (segment (start 107.455 170.32) (end 121.425 170.32) (width 2.54) (layer F.Cu) (net 7))
-  (segment (start 114.44 151.665) (end 114.44 145.555) (width 0.508) (layer F.Cu) (net 8))
+  (segment (start 113.565 152.54) (end 111.9 152.54) (width 0.3048) (layer F.Cu) (net 8))
+  (segment (start 111.9 152.54) (end 108.725 149.365) (width 0.3048) (layer F.Cu) (net 8))
+  (segment (start 108.725 149.365) (end 108.725 145.555) (width 0.3048) (layer F.Cu) (net 8))
+  (segment (start 108.09 144.92) (end 101.74 144.92) (width 0.3048) (layer F.Cu) (net 8))
+  (segment (start 108.725 145.555) (end 108.09 144.92) (width 0.3048) (layer F.Cu) (net 8))
   (segment (start 118.758 180.48) (end 118.758 181.75) (width 0.508) (layer F.Cu) (net 17))
   (segment (start 117.615 179.21) (end 118.758 180.48) (width 0.508) (layer F.Cu) (net 17))
-  (segment (start 108.725 179.21) (end 117.615 179.21) (width 0.508) (layer F.Cu) (net 17))
-  (segment (start 104.28 183.655) (end 108.725 179.21) (width 0.508) (layer F.Cu) (net 17))
-  (segment (start 90.31 183.655) (end 104.28 183.655) (width 0.508) (layer F.Cu) (net 17))
+  (segment (start 98.565 179.21) (end 117.615 179.21) (width 0.508) (layer F.Cu) (net 17))
+  (segment (start 94.12 183.655) (end 98.565 179.21) (width 0.508) (layer F.Cu) (net 17))
+  (segment (start 90.31 183.655) (end 94.12 183.655) (width 0.508) (layer F.Cu) (net 17))
   (segment (start 129.045 179.845) (end 124.727 179.845) (width 0.508) (layer F.Cu) (net 19))
   (segment (start 131.585 182.385) (end 129.045 179.845) (width 0.508) (layer F.Cu) (net 19))
@@
   (segment (start 87.77 196.355) (end 87.77 200.165) (width 0.508) (layer F.Cu) (net 19))
   (segment (start 90.31 193.815) (end 87.77 196.355) (width 0.508) (layer F.Cu) (net 19))
+  (segment (start 94.12 184.925) (end 90.31 188.735) (width 0.508) (layer F.Cu) (net 22))
+  (segment (start 98.565 180.48) (end 94.12 184.925) (width 0.508) (layer F.Cu) (net 22))
+  (segment (start 113.805 180.48) (end 98.565 180.48) (width 0.508) (layer F.Cu) (net 22))
   (segment (start 115.075 181.75) (end 113.805 180.48) (width 0.508) (layer F.Cu) (net 22))
   (segment (start 115.075 183.02) (end 115.075 181.75) (width 0.508) (layer F.Cu) (net 22))
@@
   (segment (start 121.806 184.544) (end 121.425 184.925) (width 0.508) (layer F.Cu) (net 22))
   (segment (start 121.806 183.53) (end 121.806 184.544) (width 0.508) (layer F.Cu) (net 22))
-  (segment (start 94.12 184.925) (end 90.31 188.735) (width 0.508) (layer F.Cu) (net 22))
-  (segment (start 104.28 184.925) (end 94.12 184.925) (width 0.508) (layer F.Cu) (net 22))
-  (segment (start 108.725 180.48) (end 104.28 184.925) (width 0.508) (layer F.Cu) (net 22))
-  (segment (start 113.805 180.48) (end 108.725 180.48) (width 0.508) (layer F.Cu) (net 22))
   (segment (start 123.838 183.53) (end 123.838 192.037) (width 0.508) (layer F.Cu) (net 23))
   (segment (start 123.838 192.037) (end 116.98 198.895) (width 0.508) (layer F.Cu) (net 23))
@@
     (polygon
       (pts
-        (xy 231.915 224.93) (xy 68.085 224.93) (xy 68.085 146.19) (xy 93.485 146.19) (xy 97.295 150)
-        (xy 109.36 150) (xy 110.63 148.73) (xy 110.63 141.11) (xy 111.265 141.11) (xy 122.695 141.11)
-        (xy 128.41 135.395) (xy 128.41 75.07) (xy 231.915 75.07)
+        (xy 231.915 224.93) (xy 68.085 224.93) (xy 68.085 75.07) (xy 231.915 75.07)
       )
     )
   )
   (zone (net 4) (net_name "Net-(F1-Pad2)") (layer F.Cu) (hatch edge 0.508)
+    (priority 1)
     (connect_pads yes (clearance 0.2032))
     (min_thickness 0.2032)
@@
     (polygon
       (pts
-        (xy 68.085 145.555) (xy 68.085 75.07) (xy 127.775 75.07) (xy 127.775 135.395) (xy 122.695 140.475)
-        (xy 109.995 140.475) (xy 109.995 148.73) (xy 109.36 149.365) (xy 97.295 149.365) (xy 93.485 145.555)
+        (xy 68.085 145.555) (xy 68.085 75.07) (xy 134.125 75.07) (xy 134.125 148.73) (xy 133.49 149.365)
+        (xy 120.79 149.365) (xy 120.155 148.73) (xy 120.155 141.745) (xy 118.885 140.475) (xy 97.93 140.475)
+        (xy 92.85 145.555)
       )
     )
   )
   (zone (net 11) (net_name "Net-(F3-Pad1)") (layer F.Cu) (hatch edge 0.508)
-    (priority 1)
+    (priority 2)
     (connect_pads yes (clearance 0.2032))
     (min_thickness 0.2032)
@@
   )
   (zone (net 12) (net_name "Net-(F4-Pad1)") (layer F.Cu) (hatch edge 0.508)
-    (priority 1)
+    (priority 2)
     (connect_pads yes (clearance 0.2032))
     (min_thickness 0.2032)

Commit message: Update pcb layout
Parts:
- removed H10: MountingHole, MountingHole:MountingHole_4.3mm_M4
- moved REF** 5.08 mm to (213.5, 214.1)
- moved H9 3.36 mm to (125.0, 200.0)
- moved REF** 3.18 mm to (184.9, 204.0)
- moved C6 2.62 mm to (77.0, 180.5)
- moved F4 2.54 mm to (96.7, 109.4)
- moved J4 2.54 mm to (96.7, 99.2)
- moved J8 2.54 mm to (87.8, 219.2)
Routing:
- net Net-(C6-Pad1): track 46.2 -> 43.6 mm
- net Net-(J7-Pad6): track 32.1 -> 34.7 mm
- net Net-(J7-Pad3): track 38.7 -> 41.2 mm
- net Net-(J7-Pad1): track 44.9 -> 47.2 mm
- net Net-(J7-Pad2): track 72.5 -> 73.6 mm
- net GND: vias 373 -> 339
Other:
- outline, holes or cut-outs redrawn
- board text added: "12V"
- board text added: "BK"
- board text removed: "+12V"
- board text removed: "BLACK"

Commit message: Update schematics and layout
Parts:
- removed H7, H8, H9: MountingHole, MountingHole:MountingHole_4.3mm_M4
- moved REF** 8.35 mm to (214.8, 205.9)
- moved J7 8.09 mm to (116.3, 180.5)
- moved J8 4.62 mm to (86.5, 214.8)
- moved J6 4.07 mm to (118.2, 167.8)
- moved C1 3.81 mm to (105.5, 153.8)
- moved C2 3.81 mm to (79.5, 158.3)
- moved C3 3.81 mm to (79.5, 160.8)
- moved C4 3.81 mm to (105.5, 156.3)
- moved C6 3.81 mm to (77.0, 176.7)
- moved F1 3.81 mm to (90.3, 142.4)
- moved F2 3.81 mm to (81.4, 142.4)
- moved R1 3.81 mm to (114.4, 148.7)
- moved U1 3.81 mm to (107.5, 164.0)
- moved U2 3.81 mm to (79.5, 169.1)
- moved D1 3.81 mm to (113.2, 157.0)
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Routing:
- net Net-(C1-Pad1): track 38.3 -> 0.00 mm
- net Net-(C2-Pad1): track 26.6 -> 0.00 mm
- net Net-(C5-Pad1): track 14.0 -> 0.00 mm
- net Net-(J7-Pad2): track 73.6 -> 64.8 mm
- net Net-(J7-Pad6): track 34.7 -> 27.5 mm
- net Net-(J7-Pad1): track 47.2 -> 40.5 mm
- net Net-(J7-Pad3): track 41.2 -> 35.0 mm
- net Net-(C6-Pad1): track 43.6 -> 42.5 mm
- net GND: vias 339 -> 349
- added copper zone on F.Cu, net Net-(C1-Pad1)
- added copper zone on F.Cu, net Net-(C2-Pad1)
- added copper zone on F.Cu, net Net-(C5-Pad1)
Other:
- outline, holes or cut-outs redrawn
- board text added: "BLACK"
- board text removed: "BK"
