File: perception-array-interface-box.sch (KiCad schematic (older format))
At the start: 33 parts, among them J1 PV-3, J2 PV-3, J3 PV-3, J4 2-5530843-7, J5 2-5530843-7, J6 Conn_01x02, J7 RJHSE5381, J8 1715789, U1 K7805-2000R3, U2 K7812-2000R3L

Commit message: Update pcb layout
Parts:
- removed H10: MountingHole, MountingHole:MountingHole_4.3mm_M4, symbol Mechanical:MountingHole
Changed lines of the file:
@@
-$EndComp
-$Comp
-L Mechanical:MountingHole H10
-U 1 1 60BED6D4
-P 10450 2850
-F 0 "H10" H 10550 2896 50  0000 L CNN
-F 1 "MountingHole" H 10550 2805 50  0000 L CNN
-F 2 "MountingHole:MountingHole_4.3mm_M4" H 10450 2850 50  0001 C CNN
-F 3 "~" H 10450 2850 50  0001 C CNN
-	1    10450 2850
-	1    0    0    -1
 $EndComp
 $Comp

Commit message: Update schematics and layout
Parts:
- removed H7, H8, H9: MountingHole, MountingHole:MountingHole_4.3mm_M4, symbol Mechanical:MountingHole
Changed lines of the file:
@@
 F 1 "Mini Blade Fuse 32V 3A" V 3144 2600 50  0000 C CNN
 F 2 "Fuse:RSPRO_1884617_plus_fuse" V 3180 2600 50  0001 C CNN
-F 3 "~" H 3250 2600 50  0001 C CNN
+F 3 "https://docs.rs-online.com/92e6/A700000006779340.pdf" H 3250 2600 50  0001 C CNN
 	1    3250 2600
 	0    1    1    0
@@
 F 1 "Mini Blade Fuse 32V 3A" V 3144 1500 50  0000 C CNN
 F 2 "Fuse:RSPRO_1884617_plus_fuse" V 3180 1500 50  0001 C CNN
-F 3 "~" H 3250 1500 50  0001 C CNN
+F 3 "https://docs.rs-online.com/92e6/A700000006779340.pdf" H 3250 1500 50  0001 C CNN
 	1    3250 1500
 	0    1    1    0
@@
 $EndComp
 $Comp
-L Mechanical:MountingHole H7
-U 1 1 60BECE34
-P 10450 2250
-F 0 "H7" H 10550 2296 50  0000 L CNN
-F 1 "MountingHole" H 10550 2205 50  0000 L CNN
-F 2 "MountingHole:MountingHole_4.3mm_M4" H 10450 2250 50  0001 C CNN
-F 3 "~" H 10450 2250 50  0001 C CNN
-	1    10450 2250
-	1    0    0    -1
-$EndComp
-$Comp
-L Mechanical:MountingHole H8
-U 1 1 60BED400
-P 10450 2450
-F 0 "H8" H 10550 2496 50  0000 L CNN
-F 1 "MountingHole" H 10550 2405 50  0000 L CNN
-F 2 "MountingHole:MountingHole_4.3mm_M4" H 10450 2450 50  0001 C CNN
-F 3 "~" H 10450 2450 50  0001 C CNN
-	1    10450 2450
-	1    0    0    -1
-$EndComp
-$Comp
-L Mechanical:MountingHole H9
-U 1 1 60BED565
-P 10450 2650
-F 0 "H9" H 10550 2696 50  0000 L CNN
-F 1 "MountingHole" H 10550 2605 50  0000 L CNN
-F 2 "MountingHole:MountingHole_4.3mm_M4" H 10450 2650 50  0001 C CNN
-F 3 "~" H 10450 2650 50  0001 C CNN
-	1    10450 2650
-	1    0    0    -1
-$EndComp
-$Comp
 L Device:C C1
 U 1 1 60C46DB4
@@
 F 1 "5KP30A-E3/54" V 4045 1830 50  0000 L CNN
 F 2 "Diode_THT:D_P600_R-6_P7.62mm_Vertical_KathodeUp" H 4000 1750 50  0001 C CNN
-F 3 "~" H 4000 1750 50  0001 C CNN
+F 3 "https://www.vishay.com/docs/88308/88308.pdf" H 4000 1750 50  0001 C CNN
 	1    4000 1750
 	0    1    1    0
@@
 F 1 "5KP30A-E3/54" V 4045 2930 50  0000 L CNN
 F 2 "Diode_THT:D_P600_R-6_P7.62mm_Vertical_KathodeUp" H 4000 2850 50  0001 C CNN
-F 3 "~" H 4000 2850 50  0001 C CNN
+F 3 "https://www.vishay.com/docs/88308/88308.pdf" H 4000 2850 50  0001 C CNN
 	1    4000 2850
 	0    1    1    0
@@
 F 1 "Mini Blade Fuse 32V 3A" V 3144 3500 50  0000 C CNN
 F 2 "Fuse:RSPRO_1884617_plus_fuse" V 3180 3500 50  0001 C CNN
-F 3 "~" H 3250 3500 50  0001 C CNN
+F 3 "https://docs.rs-online.com/92e6/A700000006779340.pdf" H 3250 3500 50  0001 C CNN
 	1    3250 3500
 	0    1    1    0
@@
 F 1 "Mini Blade Fuse 32V 3A" V 3144 4000 50  0000 C CNN
 F 2 "Fuse:RSPRO_1884617_plus_fuse" V 3180 4000 50  0001 C CNN
-F 3 "~" H 3250 4000 50  0001 C CNN
+F 3 "https://docs.rs-online.com/92e6/A700000006779340.pdf" H 3250 4000 50  0001 C CNN
 	1    3250 4000
 	0    1    1    0
