File: perception-array-interface-board.kicad_pcb (KiCad board)
At the start: 2 copper layers, 162 x 148 mm, 31 parts, among them J1 PV-3, J2 PV-3, J3 PV-3, J4 2-5530843-7, J5 2-5530843-7, J6 Conn_01x02, J7 RJHSE5381, J8 1715789, U1 K7805-2000R3, U2 K7812-2000R3L

Commit message: Update kicad files
Parts:
- removed the REF** at (214.8, 205.9)
- J4, J5: footprint Connector:TEConnectivity_2-5530843-7 -> Connector:TE-Connectivity_2-5530843-7
- U1: footprint SuperRegulator:K78xx-2000R3 -> SuperRegulator:RSPRO_K78xx-2000R3
- U2: footprint SuperRegulator:K78xx-2000R3L -> SuperRegulator:RSPRO_K78xx-2000R3L

Commit message: Update kicad files
Connections:
- J4 pad 1: GND -> Net-(J4-Pad1)
- J4 pad 3: GND -> Net-(J4-Pad3)
- J4 pad 32: GND -> Net-(J4-Pad32)
- J4 pad 34: GND -> Net-(J4-Pad34)
- J4 pad 36: GND -> Net-(J4-Pad36)
- J4 pad 5: GND -> Net-(J4-Pad5)
- J5 pad 1: GND -> Net-(J5-Pad1)
- J5 pad 3: GND -> Net-(J5-Pad3)
- J5 pad 32: GND -> Net-(J5-Pad32)
- J5 pad 34: GND -> Net-(J5-Pad34)
- J5 pad 36: GND -> Net-(J5-Pad36)
- J5 pad 5: GND -> Net-(J5-Pad5)
Routing:
- net GND: vias 349 -> 348
Other:
- outline, holes or cut-outs redrawn

Commit message: Update kicad files
Parts:
- added J7: Conn_01x01, Connector_Pin:Pin_D1.4mm_L8.5mm_W2.8mm_FlatFork, F.Cu at (122.7, 167.8)
- J6: value Conn_01x02 -> Conn_01x01; footprint Connector_PinHeader_2.54mm:PinHeader_1x02_P2.54mm_Vertical -> Connector_Pin:Pin_D1.4mm_L8.5mm_W2.8mm_FlatFork
- moved J6 0.64 mm to (117.6, 167.8), turned to 0 degrees
- renumbered J7 to J8, J8 to J9
