File: perception-array-interface-board.sch (KiCad schematic (older format))
At the start: 29 parts, among them J1 PV-3, J2 PV-3, J3 PV-3, J4 2-5530843-7, J5 2-5530843-7, J6 Conn_01x02, J7 RJHSE5381, J8 1715789, U1 K7805-2000R3, U2 K7812-2000R3L

Commit message: Update kicad files
Parts:
- J4, J5: footprint Connector:TEConnectivity_2-5530843-7 -> Connector:TE-Connectivity_2-5530843-7
- U1: footprint SuperRegulator:K78xx-2000R3 -> SuperRegulator:RSPRO_K78xx-2000R3
- U2: footprint SuperRegulator:K78xx-2000R3L -> SuperRegulator:RSPRO_K78xx-2000R3L
Changed lines of the file:
@@
 encoding utf-8
 Sheet 1 1
-Title ""
-Date ""
+Title "Perception Array Interface Board"
+Date "2021-07-10"
 Rev ""
-Comp ""
+Comp "OUXT Polaris"
 Comment1 ""
 Comment2 ""
@@
 F 0 "U1" H 6250 1742 50  0000 C CNN
 F 1 "K7805-2000R3" H 6250 1651 50  0000 C CNN
-F 2 "SuperRegulator:K78xx-2000R3" H 6250 1725 50  0001 C CIN
+F 2 "SuperRegulator:RSPRO_K78xx-2000R3" H 6250 1725 50  0001 C CIN
 F 3 "https://docs.rs-online.com/fc3c/A700000006631878.pdf" H 6250 1450 50  0001 C CNN
 	1    6250 1500
@@
 F 0 "U2" H 6250 2842 50  0000 C CNN
 F 1 "K7812-2000R3L" H 6250 2751 50  0000 C CNN
-F 2 "SuperRegulator:K78xx-2000R3L" H 6250 2825 50  0001 C CIN
+F 2 "SuperRegulator:RSPRO_K78xx-2000R3L" H 6250 2825 50  0001 C CIN
 F 3 "https://docs.rs-online.com/fc3c/A700000006631878.pdf" H 6250 2550 50  0001 C CNN
 	1    6250 2600
@@
 F 0 "J5" H 6450 5667 50  0000 C CNN
 F 1 "2-5530843-7" H 6450 5576 50  0000 C CNN
-F 2 "Connector:TEConnectivity_2-5530843-7" H 6400 4650 50  0001 C CNN
+F 2 "Connector:TE-Connectivity_2-5530843-7" H 6400 4650 50  0001 C CNN
 F 3 "~" H 6400 4650 50  0001 C CNN
 	1    6400 4650
@@
 F 0 "J4" H 4950 6167 50  0000 C CNN
 F 1 "2-5530843-7" H 4950 6076 50  0000 C CNN
-F 2 "Connector:TEConnectivity_2-5530843-7" H 4900 5150 50  0001 C CNN
+F 2 "Connector:TE-Connectivity_2-5530843-7" H 4900 5150 50  0001 C CNN
 F 3 "~" H 4900 5150 50  0001 C CNN
 	1    4900 5150

Commit message: Update kicad files
Connections:
- net GND: no longer J4.1 (Pin_1), J4.3 (Pin_3), J4.32 (Pin_32), J4.34 (Pin_34), J4.36 (Pin_36), J4.5 (Pin_5), J5.1 (Pin_1), J5.3 (Pin_3), J5.32 (Pin_32), J5.34 (Pin_34), J5.36 (Pin_36), J5.5 (Pin_5)
- no-connect marks 0 -> 12
Changed lines of the file:
@@
 	1700 1500 2500 1500
 Connection ~ 2500 1500
-Wire Wire Line
-	4400 4350 4400 4450
 $Comp
 L power:GND #PWR05
@@
 Wire Wire Line
 	4400 4750 4400 4850
-Connection ~ 4400 4650
 Wire Wire Line
 	4400 4650 4400 4750
-Wire Wire Line
-	4600 4550 4400 4550
-Connection ~ 4400 4550
-Wire Wire Line
-	4400 4550 4400 4650
-Connection ~ 4400 4450
-Wire Wire Line
-	4400 4450 4400 4550
 $Comp
 L Connector:8P8C_LED_Shielded J7
@@
 	5200 5050 5200 4000
 Connection ~ 5200 5050
-$Comp
-L Connector_Generic:Conn_02x18_Odd_Even J5
-U 1 1 60C91187
-P 6400 4650
-F 0 "J5" H 6450 5667 50  0000 C CNN
-F 1 "2-5530843-7" H 6450 5576 50  0000 C CNN
-F 2 "Connector:TE-Connectivity_2-5530843-7" H 6400 4650 50  0001 C CNN
-F 3 "~" H 6400 4650 50  0001 C CNN
-	1    6400 4650
-	-1   0    0    -1
-$EndComp
 $Comp
 L Device:C C1
@@
 	4400 4950 4400 5450
 Wire Wire Line
-	4400 4350 4600 4350
-Wire Wire Line
-	4400 4450 4600 4450
-Wire Wire Line
 	4400 4650 4600 4650
 $Comp
 L Connector_Generic:Conn_02x18_Odd_Even J4
 U 1 1 60C8DD8E
-P 4900 5150
-F 0 "J4" H 4950 6167 50  0000 C CNN
-F 1 "2-5530843-7" H 4950 6076 50  0000 C CNN
-F 2 "Connector:TE-Connectivity_2-5530843-7" H 4900 5150 50  0001 C CNN
-F 3 "~" H 4900 5150 50  0001 C CNN
-	1    4900 5150
-	-1   0    0    -1
+P 4800 5150
+F 0 "J4" H 4850 6167 50  0000 C CNN
+F 1 "2-5530843-7" H 4850 6076 50  0000 C CNN
+F 2 "Connector:TE-Connectivity_2-5530843-7" H 4800 5150 50  0001 C CNN
+F 3 "~" H 4800 5150 50  0001 C CNN
+	1    4800 5150
+	1    0    0    -1
 $EndComp
 Wire Wire Line
@@
 	-1   0    0    -1
 $EndComp
-Connection ~ 5300 6050
-Wire Wire Line
-	5300 6050 5300 6150
-Connection ~ 5300 5950
-Wire Wire Line
-	5300 5950 5300 6050
-Connection ~ 5300 5850
-Wire Wire Line
-	5300 5850 5300 5950
 Connection ~ 5300 5750
-Wire Wire Line
-	5300 5750 5300 5850
 Connection ~ 5300 5650
 Wire Wire Line
@@
 Wire Wire Line
 	5300 5750 5100 5750
-Wire Wire Line
-	5300 5850 5100 5850
-Wire Wire Line
-	5300 5950 5100 5950
-Wire Wire Line
-	5300 6050 5100 6050
-Wire Wire Line
-	5900 3850 5900 3950
 $Comp
 L power:GND #PWR011
@@
 Wire Wire Line
 	5900 4250 5900 4350
-Connection ~ 5900 4150
 Wire Wire Line
 	5900 4150 5900 4250
-Wire Wire Line
-	6100 4050 5900 4050
-Connection ~ 5900 4050
-Wire Wire Line
-	5900 4050 5900 4150
-Connection ~ 5900 3950
-Wire Wire Line
-	5900 3950 5900 4050
 Wire Wire Line
 	6100 4550 6000 4550
@@
 	5900 4450 5900 4950
 Wire Wire Line
-	5900 3850 6100 3850
-Wire Wire Line
-	5900 3950 6100 3950
-Wire Wire Line
 	5900 4150 6100 4150
 Wire Wire Line
@@
 Wire Wire Line
 	6700 4650 6700 4750
-Wire Wire Line
-	6700 4550 6700 3500
 Connection ~ 6700 4550
 Wire Wire Line
@@
 	-1   0    0    -1
 $EndComp
-Connection ~ 6800 5550
-Wire Wire Line
-	6800 5550 6800 5650
-Connection ~ 6800 5450
-Wire Wire Line
-	6800 5450 6800 5550
-Connection ~ 6800 5350
-Wire Wire Line
-	6800 5350 6800 5450
 Connection ~ 6800 5250
-Wire Wire Line
-	6800 5250 6800 5350
 Connection ~ 6800 5150
 Wire Wire Line
@@
 Wire Wire Line
 	6800 4150 6800 4250
-Wire Wire Line
-	6600 4050 6800 4050
 Connection ~ 6800 4050
 Wire Wire Line
@@
 Wire Wire Line
 	6800 4450 6800 4950
-Wire Wire Line
-	6800 3850 6600 3850
-Wire Wire Line
-	6800 3950 6600 3950
-Wire Wire Line
-	6800 4150 6600 4150
-Wire Wire Line
-	6800 4250 6600 4250
-Wire Wire Line
-	6800 4350 6600 4350
-Wire Wire Line
-	6800 4450 6600 4450
-Wire Wire Line
-	6800 4950 6600 4950
-Wire Wire Line
-	6800 5050 6600 5050
-Wire Wire Line
-	6800 5150 6600 5150
-Wire Wire Line
-	6800 5250 6600 5250
-Wire Wire Line
-	6800 5350 6600 5350
-Wire Wire Line
-	6800 5450 6600 5450
-Wire Wire Line
-	6800 5550 6600 5550
 Wire Wire Line
 	6000 3500 6700 3500
@@
 Wire Wire Line
 	9000 2600 9000 4050
+Wire Wire Line
+	6800 4150 6600 4150
+Wire Wire Line
+	6600 4050 6800 4050
+Wire Wire Line
+	6800 3950 6600 3950
+Wire Wire Line
+	6800 5250 6600 5250
+Wire Wire Line
+	6800 5150 6600 5150
+Wire Wire Line
+	6800 5050 6600 5050
+Wire Wire Line
+	6800 4950 6600 4950
+Wire Wire Line
+	6800 3850 6600 3850
+Wire Wire Line
+	6800 4450 6600 4450
+Wire Wire Line
+	6800 4350 6600 4350
+Wire Wire Line
+	6800 4250 6600 4250
+Wire Wire Line
+	6700 4550 6700 3500
+$Comp
+L Connector_Generic:Conn_02x18_Odd_Even J5
+U 1 1 60C91187
+P 6300 4650
+F 0 "J5" H 6350 5667 50  0000 C CNN
+F 1 "2-5530843-7" H 6350 5576 50  0000 C CNN
+F 2 "Connector:TE-Connectivity_2-5530843-7" H 6300 4650 50  0001 C CNN
+F 3 "~" H 6300 4650 50  0001 C CNN
+	1    6300 4650
+	1    0    0    -1
+$EndComp
+Wire Wire Line
+	5300 5750 5300 6150
+Wire Wire Line
+	6800 5250 6800 5650
+NoConn ~ 6600 5350
+NoConn ~ 6600 5450
+NoConn ~ 6600 5550
+NoConn ~ 5100 5850
+NoConn ~ 5100 5950
+NoConn ~ 5100 6050
+NoConn ~ 6100 3850
+NoConn ~ 4600 4350
+NoConn ~ 4600 4450
+NoConn ~ 4600 4550
+NoConn ~ 6100 3950
+NoConn ~ 6100 4050
 $EndSCHEMATC

Commit message: Update kicad files
Parts:
- removed J6: Conn_01x02, Connector_PinHeader_2.54mm:PinHeader_1x02_P2.54mm_Vertical, symbol Connector_Generic:Conn_01x02
- added J6, J7: Conn_01x01, Connector_Pin:Pin_D1.4mm_L8.5mm_W2.8mm_FlatFork, symbol Connector_Generic:Conn_01x01
- renumbered J7 to J8, J8 to J9
Connections:
- net GND: now also J7.1 (Pin_1)
- net at C5.1, U1.3 (VO): now also J6.1 (Pin_1)
Changed lines of the file:
@@
 L power:GND #PWR017
 U 1 1 60B57428
-P 7550 1700
-F 0 "#PWR017" H 7550 1450 50  0001 C CNN
-F 1 "GND" H 7555 1527 50  0000 C CNN
-F 2 "" H 7550 1700 50  0001 C CNN
-F 3 "" H 7550 1700 50  0001 C CNN
-	1    7550 1700
-	1    0    0    -1
-$EndComp
-Wire Wire Line
-	7550 1700 7550 1600
-Wire Wire Line
-	7550 1600 7650 1600
+P 7550 1800
+F 0 "#PWR017" H 7550 1550 50  0001 C CNN
+F 1 "GND" H 7555 1627 50  0000 C CNN
+F 2 "" H 7550 1800 50  0001 C CNN
+F 3 "" H 7550 1800 50  0001 C CNN
+	1    7550 1800
+	1    0    0    -1
+$EndComp
+Wire Wire Line
+	7550 1800 7550 1700
+Wire Wire Line
+	7550 1700 7650 1700
 Wire Wire Line
 	6250 1800 6250 2000
 Wire Wire Line
 	6250 2900 6250 3100
-$Comp
-L Connector_Generic:Conn_01x02 J6
-U 1 1 60B67FF9
-P 7850 1500
-F 0 "J6" H 7930 1492 50  0000 L CNN
-F 1 "Conn_01x02" H 7930 1401 50  0000 L CNN
-F 2 "Connector_PinHeader_2.54mm:PinHeader_1x02_P2.54mm_Vertical" H 7850 1500 50  0001 C CNN
-F 3 "~" H 7850 1500 50  0001 C CNN
-	1    7850 1500
-	1    0    0    -1
-$EndComp
 $Comp
 L Device:C C4
@@
 	5600 2000 5600 1900
 $Comp
-L Connector:Screw_Terminal_01x08 J8
+L Connector:Screw_Terminal_01x08 J9
 U 1 1 60B9B09F
 P 9300 3850
-F 0 "J8" H 9218 3225 50  0000 C CNN
+F 0 "J9" H 9218 3225 50  0000 C CNN
 F 1 "1715789" H 9218 3316 50  0000 C CNN
 F 2 "TerminalBlock_Phoenix:TerminalBlock_Phoenix_MKDS-1,5-8-5.08_1x08_P5.08mm_Horizontal" H 9300 3850 50  0001 C CNN
@@
 	4400 4650 4400 4750
 $Comp
-L Connector:8P8C_LED_Shielded J7
+L Connector:8P8C_LED_Shielded J8
 U 1 1 60BDC610
 P 8100 3650
-F 0 "J7" H 8100 4317 50  0000 C CNN
+F 0 "J8" H 8100 4317 50  0000 C CNN
 F 1 "RJHSE5381" H 8100 4226 50  0000 C CNN
 F 2 "Connector_RJ:RJ45_Amphenol_RJHSE538X" V 8100 3675 50  0001 C CNN
@@
 NoConn ~ 6100 3950
 NoConn ~ 6100 4050
+$Comp
+L Connector_Generic:Conn_01x01 J6
+U 1 1 6111C44D
+P 7850 1500
+F 0 "J6" H 7930 1542 50  0000 L CNN
+F 1 "Conn_01x01" H 7930 1451 50  0000 L CNN
+F 2 "Connector_Pin:Pin_D1.4mm_L8.5mm_W2.8mm_FlatFork" H 7850 1500 50  0001 C CNN
+F 3 "~" H 7850 1500 50  0001 C CNN
+	1    7850 1500
+	1    0    0    -1
+$EndComp
+$Comp
+L Connector_Generic:Conn_01x01 J7
+U 1 1 6111C952
+P 7850 1700
+F 0 "J7" H 7930 1742 50  0000 L CNN
+F 1 "Conn_01x01" H 7930 1651 50  0000 L CNN
+F 2 "Connector_Pin:Pin_D1.4mm_L8.5mm_W2.8mm_FlatFork" H 7850 1700 50  0001 C CNN
+F 3 "~" H 7850 1700 50  0001 C CNN
+	1    7850 1700
+	1    0    0    -1
+$EndComp
 $EndSCHEMATC
